File: router/router.brd (EAGLE design)
At the start: 49.5 x 47.6 mm, 20 parts, among them IC1 REG1117, J1 nRF24, J4 6_PIN_SERIAL_CABLEPTH, J5 POWER_JACKSLT

Commit message: Double-sided Node Trial Run v0.3b
Connections:
- new net N$1: R5.1
- net GND: no longer R5.1
Changed lines of the file:
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@@
 <contactref element="C5" pad="2"/>
 <contactref element="J1" pad="1"/>
-<contactref element="J2" pad="8"/>
-<contactref element="R5" pad="1"/>
 <contactref element="J3" pad="GND"/>
 <polygon width="0.1524" layer="1">
@@
 <wire x1="-8.5725" y1="-2.2225" x2="-8.5725" y2="-11.1125" width="0.1524" layer="16"/>
 <wire x1="-8.5725" y1="-11.1125" x2="-8.89" y2="-11.43" width="0.1524" layer="16"/>
+<contactref element="J2" pad="8"/>
 </signal>
 <signal name="RST">
@@
 </polygon>
 </signal>
+<signal name="N$1">
+<contactref element="R5" pad="1"/>
+</signal>
 </signals>
