File: router/router.sch (EAGLE design)
At the start: 20 parts, among them IC1 REG1117, J1 nRF24, J4 6_PIN_SERIAL_CABLEPTH, J5 POWER_JACKSLT

Commit message: Double-sided Node Trial Run v0.3b
Connections:
- new net N$1: R5.1
- net GND: no longer R5.1
Changed lines of the file:
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@@
 <part name="J5" library="SparkFun-Connectors" deviceset="POWER_JACK" device="SLT"/>
 <part name="IC1" library="burr-brown" library_urn="urn:adsk.eagle:library:111" deviceset="REG1117" device="" package3d_urn="urn:adsk.eagle:package:4940/1"/>
+<part name="GND11" library="SparkFun-PowerSymbols" deviceset="GND" device=""/>
 </parts>
 <sheets>
@@
 <instance part="J5" gate="G$1" x="116.84" y="-33.02"/>
 <instance part="IC1" gate="G$1" x="116.84" y="-48.26"/>
+<instance part="GND11" gate="1" x="111.76" y="-10.16"/>
 </instances>
 <busses>
@@
 </segment>
 <segment>
-<pinref part="J2" gate="G$1" pin="8"/>
-<label x="109.22" y="-10.16" size="1.778" layer="95"/>
-<pinref part="R5" gate="G$1" pin="1"/>
-<wire x1="101.6" y1="-5.08" x2="99.06" y2="-5.08" width="0.1524" layer="91"/>
-<wire x1="99.06" y1="-5.08" x2="99.06" y2="-7.62" width="0.1524" layer="91"/>
-<wire x1="99.06" y1="-7.62" x2="111.76" y2="-7.62" width="0.1524" layer="91"/>
-</segment>
-<segment>
 <pinref part="GND9" gate="1" pin="GND"/>
 <wire x1="15.24" y1="-35.56" x2="15.24" y2="-33.02" width="0.1524" layer="91"/>
@@
 <junction x="119.38" y="-30.48"/>
 <junction x="119.38" y="-27.94"/>
+</segment>
+<segment>
+<pinref part="J2" gate="G$1" pin="8"/>
+<pinref part="GND11" gate="1" pin="GND"/>
 </segment>
 </net>
@@
 </segment>
 </net>
+<net name="N$1" class="0">
+<segment>
+<pinref part="R5" gate="G$1" pin="1"/>
+<wire x1="101.6" y1="-5.08" x2="101.6" y2="-2.54" width="0.1524" layer="91"/>
+<wire x1="101.6" y1="-2.54" x2="109.22" y2="-2.54" width="0.1524" layer="91"/>
+</segment>
+</net>
