File: sensor-template/sensor-dht-volt-generic.brd (EAGLE design)
At the start: 22.1 x 27.3 mm, 19 parts, among them U2 ATMEGA328PB-AUR

Commit message: [sensor] Debug connector now complies to node arrangement
Connections:
- net RX0: now also DEBUG.3; no longer DEBUG.4
- net TX0: now also DEBUG.4; no longer DEBUG.3
Routing:
- net RX0: track 3.27 -> 7.00 mm
- net TX0: track 6.14 -> 3.61 mm
Changed lines of the file:
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@@
 <signal name="RX0">
 <contactref element="U2" pad="30"/>
-<contactref element="DEBUG" pad="4"/>
-<wire x1="13.8982" y1="15.4497" x2="16.474790625" y2="15.4497" width="0.1524" layer="16"/>
-<wire x1="16.474790625" y1="15.4497" x2="16.65439375" y2="15.52409375" width="0.1524" layer="16" curve="44.999502"/>
-<wire x1="16.65439375" y1="15.52409375" x2="17.0053" y2="15.875" width="0.1524" layer="16"/>
+<contactref element="DEBUG" pad="3"/>
+<wire x1="19.12" y1="15.4497" x2="19.5453" y2="15.875" width="0.1524" layer="16"/>
+<wire x1="16.594975" y1="16.8656" x2="17.415625" y2="16.8656" width="0.1524" layer="16"/>
+<wire x1="13.8982" y1="15.4497" x2="15.179075" y2="15.4497" width="0.1524" layer="16"/>
+<wire x1="18.831525" y1="15.4497" x2="19.12" y2="15.4497" width="0.1524" layer="16"/>
+<wire x1="15.179075" y1="15.4497" x2="16.594975" y2="16.8656" width="0.1524" layer="16"/>
+<wire x1="17.415625" y1="16.8656" x2="18.831525" y2="15.4497" width="0.1524" layer="16"/>
 </signal>
 <signal name="TX0">
 <contactref element="U2" pad="31"/>
-<contactref element="DEBUG" pad="3"/>
-<wire x1="13.8982" y1="14.6497" x2="18.214790625" y2="14.6497" width="0.1524" layer="16"/>
-<wire x1="18.214790625" y1="14.6497" x2="18.39439375" y2="14.72409375" width="0.1524" layer="16" curve="44.999502"/>
-<wire x1="18.39439375" y1="14.72409375" x2="19.5453" y2="15.875" width="0.1524" layer="16"/>
+<contactref element="DEBUG" pad="4"/>
+<wire x1="13.8982" y1="14.6497" x2="15.78" y2="14.6497" width="0.1524" layer="16"/>
+<wire x1="15.78" y1="14.6497" x2="17.0053" y2="15.875" width="0.1524" layer="16"/>
 </signal>
 <signal name="N$1">
