File: sensor-template/sensor-i2c-proto.sch (EAGLE design)
At the start: 14 parts, among them U2 ATMEGA328PB-AUR

Commit message: [sensor] Debug connector now complies to node arrangement
Connections:
- net RX0: now also DEBUG.3; no longer DEBUG.4
- net TX0: now also DEBUG.4; no longer DEBUG.3
Changed lines of the file:
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@@
 </segment>
 <segment>
-<pinref part="DEBUG" gate="A" pin="4"/>
-<wire x1="177.8" y1="12.7" x2="182.88" y2="12.7" width="0.1524" layer="91"/>
-<label x="177.8" y="12.7" size="1.778" layer="95" rot="R180"/>
+<pinref part="DEBUG" gate="A" pin="3"/>
+<wire x1="195.58" y1="12.7" x2="190.5" y2="12.7" width="0.1524" layer="91"/>
+<label x="195.58" y="12.7" size="1.778" layer="95"/>
 </segment>
 </net>
@@
 </segment>
 <segment>
-<pinref part="DEBUG" gate="A" pin="3"/>
-<wire x1="195.58" y1="12.7" x2="190.5" y2="12.7" width="0.1524" layer="91"/>
-<label x="195.58" y="12.7" size="1.778" layer="95"/>
+<pinref part="DEBUG" gate="A" pin="4"/>
+<wire x1="177.8" y1="12.7" x2="182.88" y2="12.7" width="0.1524" layer="91"/>
+<label x="177.8" y="12.7" size="1.778" layer="95" rot="R180"/>
 </segment>
 </net>
