File: sensor-template/sensor-dht-volt-generic.sch (EAGLE design)
At the start: 19 parts, among them U2 ATMEGA328PB-AUR

Commit message: [sensor] Debug connector now complies to node arrangement
Connections:
- net RX0: now also DEBUG.3; no longer DEBUG.4
- net TX0: now also DEBUG.4; no longer DEBUG.3
Changed lines of the file:
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@@
 </segment>
 <segment>
-<pinref part="DEBUG" gate="A" pin="4"/>
-<wire x1="177.8" y1="12.7" x2="182.88" y2="12.7" width="0.1524" layer="91"/>
-<label x="177.8" y="12.7" size="1.778" layer="95" rot="R180"/>
+<pinref part="DEBUG" gate="A" pin="3"/>
+<wire x1="195.58" y1="12.7" x2="190.5" y2="12.7" width="0.1524" layer="91"/>
+<label x="195.58" y="12.7" size="1.778" layer="95"/>
 </segment>
 </net>
@@
 </segment>
 <segment>
-<pinref part="DEBUG" gate="A" pin="3"/>
-<wire x1="195.58" y1="12.7" x2="190.5" y2="12.7" width="0.1524" layer="91"/>
-<label x="195.58" y="12.7" size="1.778" layer="95"/>
+<pinref part="DEBUG" gate="A" pin="4"/>
+<wire x1="177.8" y1="12.7" x2="182.88" y2="12.7" width="0.1524" layer="91"/>
+<label x="177.8" y="12.7" size="1.778" layer="95" rot="R180"/>
 </segment>
 </net>

Commit message: Optional pullup on I2C + Default I2C0
Parts:
- removed C5: 10u, resistor:C-USC0603
- removed C6: 0.1u, resistor:C-USC0603
- added J_SCL: SCL_Select, SparkFun-Jumpers:JUMPER-SMT_3_1-NC_TRACE_SILK
- added J_SDA: SDA_Select, SparkFun-Jumpers:JUMPER-SMT_3_1-NC_TRACE_SILK
- added R6, R7: 10k, resistor:R-US_R0603
Connections:
- new net SCL: J_SCL.2, R6.2, U$3.4, U$4.4
- new net SDA: J_SDA.2, R7.2, U$3.3, U$4.3
- net SCL0: now also J_SCL.3
- net SCL1: now also J_SCL.1; no longer U$3.4, U$4.4
- net SDA0: now also J_SDA.3
- net SDA1: now also J_SDA.1; no longer U$3.3, U$4.3
- net VCC: now also R6.1, R7.1; no longer C5.1, C6.1
