File: Weigh_scale1.sch (EAGLE design)
At the start: 4 parts

Commit message: Add files via upload
Parts:
- added SV3, SV4: (no value), con-lstb:MA03-1
Connections:
- removed net HX_SCK: SV1.3
- new net HX_SCK_A2: SV1.3, SV3.2
- net GND: now also SV3.3
- net HX_DATA: now also SV4.1
- net VCC: now also SV3.1
Changed lines of the file:
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@@
 <part name="GND2" library="supply1" library_urn="urn:adsk.eagle:library:371" deviceset="GND" device=""/>
 <part name="L_IN" library="con-tycoelectronics" library_urn="urn:adsk.eagle:library:193" deviceset="RJ45*2" device="-B" package3d_urn="urn:adsk.eagle:package:10664/1" technology="-6L" value="flip"/>
+<part name="SV3" library="con-lstb" library_urn="urn:adsk.eagle:library:162" deviceset="MA03-1" device="" package3d_urn="urn:adsk.eagle:package:8339/1"/>
+<part name="SV4" library="con-lstb" library_urn="urn:adsk.eagle:library:162" deviceset="MA03-1" device="" package3d_urn="urn:adsk.eagle:package:8339/1"/>
 </parts>
 <sheets>
@@
 <attribute name="VALUE" x="20.32" y="22.86" size="1.778" layer="96" rot="MR90"/>
 </instance>
+<instance part="SV3" gate="G$1" x="137.16" y="53.34" smashed="yes" rot="R180">
+<attribute name="VALUE" x="138.43" y="60.96" size="1.778" layer="96" rot="R180"/>
+<attribute name="NAME" x="138.43" y="47.498" size="1.778" layer="95" rot="R180"/>
+</instance>
+<instance part="SV4" gate="G$1" x="137.16" y="35.56" smashed="yes" rot="R180">
+<attribute name="VALUE" x="138.43" y="43.18" size="1.778" layer="96" rot="R180"/>
+<attribute name="NAME" x="138.43" y="29.718" size="1.778" layer="95" rot="R180"/>
+</instance>
 </instances>
 <busses>
@@
 <pinref part="SV1" gate="1" pin="4"/>
 <pinref part="P+1" gate="VCC" pin="VCC"/>
+<pinref part="SV3" gate="G$1" pin="1"/>
+<wire x1="104.14" y1="55.88" x2="129.54" y2="55.88" width="0.1524" layer="91"/>
+<junction x="104.14" y="55.88"/>
 </segment>
 </net>
@@
 <pinref part="SV1" gate="1" pin="1"/>
 <pinref part="GND2" gate="1" pin="GND"/>
+<pinref part="SV3" gate="G$1" pin="3"/>
+<wire x1="104.14" y1="48.26" x2="129.54" y2="48.26" width="0.1524" layer="91"/>
+<wire x1="129.54" y1="48.26" x2="129.54" y2="50.8" width="0.1524" layer="91"/>
+<junction x="104.14" y="48.26"/>
 </segment>
 </net>
-<net name="HX_SCK" class="0">
+<net name="HX_SCK_A2" class="0">
 <segment>
 <pinref part="SV1" gate="1" pin="3"/>
-<wire x1="104.14" y1="53.34" x2="119.38" y2="53.34" width="0.1524" layer="91"/>
+<wire x1="104.14" y1="53.34" x2="129.54" y2="53.34" width="0.1524" layer="91"/>
 <label x="109.22" y="53.34" size="1.778" layer="95"/>
+<pinref part="SV3" gate="G$1" pin="2"/>
 </segment>
 </net>
@@
 <segment>
 <pinref part="SV1" gate="1" pin="2"/>
-<wire x1="104.14" y1="50.8" x2="119.38" y2="50.8" width="0.1524" layer="91"/>
+<wire x1="104.14" y1="50.8" x2="124.46" y2="50.8" width="0.1524" layer="91"/>
 <label x="109.22" y="50.8" size="1.778" layer="95"/>
+<wire x1="124.46" y1="50.8" x2="124.46" y2="38.1" width="0.1524" layer="91"/>
+<pinref part="SV4" gate="G$1" pin="1"/>
+<wire x1="124.46" y1="38.1" x2="129.54" y2="38.1" width="0.1524" layer="91"/>
 </segment>
 </net>
